File: LIC_rack_ZR-00.brd (EAGLE design)
At the start: 90 x 90.8 mm, 27 parts, among them IC1 ATMEGA644A, IC2 MAX481CSA

Commit message: Dalsi upravy
Pridan mikrokontrolér a další řídící prvky ještě je nutné přidat
DMMT5401 a DMG2305UX proti přepólování
Parts:
- added C11: 10n, #PaJa_31:1206
- added C12, C13: 100n, #PaJa_31:1206
- added C14: 10u/16V, #PaJa_31:1206
- added IC3: FT232RL, ftdichip:SSOP28
- added LED1, LED2: LED_F1345PLD2-3B, LED_Knihovna:LED_F1345PLD2-3B
- added OK1, OK2, OK5: 6N137, optocoupler:DIL08
- added OK3, OK4: PC817, optocoupler:DIL04
- added R10, R11, R6, R7: 1k, #PaJa_31:1206
- added R12, R13: 580R, #PaJa_31:1206
- added R14: 10M, #PaJa_31:1206
- added R4, R5, R8: 330R, #PaJa_31:1206
- added R9: 10k, #PaJa_31:1206
- added X1: MINI-USB-SCHIELD-32005-201, con-cypressindustries:32005-201
- C10, C9: value (none) -> 22pF
- Q1: value (none) -> 14.7456MHz
- moved U$1 197.8 mm to (75.4, 29.1), turned to 270 degrees
- moved U$2 178.3 mm to (20.2, 53.8), turned to 90 degrees
- moved Q1 170.9 mm to (37.0, 50.1), turned to 270 degrees
- moved IC1 153.4 mm to (50.2, 51.7)
- moved DC1 107.9 mm to (18.3, 77.4), turned to 180 degrees
- moved DC2 107.5 mm to (10.2, 77.3), turned to 180 degrees
Connections:
- removed net VCC: IC2.8
- new net 0V: IC2.5
- new net GNDINT: C11.1, C12.1, C13.1, C14.1, IC3.18, IC3.21, IC3.25, IC3.26, IC3.7, OK2.5, OK4.3, R14.1, X1.5, X1.M1, X1.M2, X1.M3, X1.M4
- new net N$10: IC3.23, R10.1
- new net N$11: IC3.22, R11.1
- new net N$12: OK5.2, R5.2
- new net N$13: OK3.2, R10.2
- new net N$14: OK4.2, R11.2
- new net N$15: OK3.4, R12.1
- new net N$16: LED1.1K, R12.2
- new net N$17: LED2.1K, R13.2
- new net N$18: OK4.4, R13.1
- new net N$22: C12.2, IC3.17
- new net N$3: IC3.2, OK5.3
- new net N$5: OK1.2, R4.2
- new net N$6: IC3.1, OK1.3
- new net N$8: IC3.5, OK2.6, R6.1
- new net N$9: OK2.2, R8.1
- new net N.C.: X1.4
- new net RESET_AVR: OK5.6, R9.2
- new net RX_AVR: OK1.6, R7.1
- new net TX_AVR: OK2.3
- new net USB_DATA+: IC3.15, X1.3
- new net USB_DATA-: IC3.16, X1.2
- new net VCCINT: C11.2, C13.2, C14.2, IC3.20, IC3.4, OK2.7, OK2.8, OK3.1, OK4.1, R4.1, R5.1, R6.2, X1.1
- net +5V: now also IC2.8, LED1.1A, LED2.1A, OK1.7, OK1.8, OK5.7, OK5.8, R7.2, R8.2, R9.1
- net GND: now also OK1.5, OK3.3, OK5.5, R14.2; no longer IC2.5
