File: LIC_rack_ZR-00.sch (EAGLE design)
At the start: 27 parts, among them IC1 ATMEGA644A, IC2 MAX481CSA

Commit message: Dalsi upravy
Pridan mikrokontrolér a další řídící prvky ještě je nutné přidat
DMMT5401 a DMG2305UX proti přepólování
Parts:
- added C11: 10n, #PaJa_31:C-KER_1206
- added C12, C13: 100n, #PaJa_31:C-KER_1206
- added C14: 10u/16V, #PaJa_31:C-KER_1206
- added IC3: FT232RL, ftdichip:FT232RL
- added LED1, LED2: LED_F1345PLD2-3B, LED_Knihovna:LED_F1345PLD2-3B
- added OK1, OK2, OK5: 6N137, optocoupler:6N137
- added OK3, OK4: PC817, optocoupler:PC817
- added R10, R11, R6, R7: 1k, #PaJa_31:R_1206
- added R12, R13: 580R, #PaJa_31:R_1206
- added R14: 10M, #PaJa_31:R_1206
- added R4, R5, R8: 330R, #PaJa_31:R_1206
- added R9: 10k, #PaJa_31:R_1206
- added X1: MINI-USB-SCHIELD-32005-201, con-cypressindustries:MINI-USB-SCHIELD-32005-201
- C10, C9: value (none) -> 22pF
- Q1: value (none) -> 14.7456MHz
Connections:
- new net 0V: IC2P.GND
- new net GNDINT: C11.1, C12.1, C13.1, C14.1, IC3.GND, IC3.GND@1, IC3.GND@2, IC3.GND@A, IC3.TEST, OK2.GND, OK4.EMIT, R14.1, X1G$1.5, X1S.S1, X1S.S2, X1S.S3, X1S.S4
- new net N$10: IC3.CBUS0, R10.1
- new net N$11: IC3.CBUS1, R11.1
- new net N$12: OK5.A, R5.2
- new net N$13: OK3.C, R10.2
- new net N$14: OK4.C, R11.2
- new net N$15: OK3.COL, R12.1
- new net N$16: LED1_BOTTOM.C, R12.2
- new net N$17: LED2_BOTTOM.C, R13.2
- new net N$18: OK4.COL, R13.1
- new net N$22: C12.2, IC3.3V3OUT
- new net N$3: IC3.!DTR, OK5.C
- new net N$5: OK1.A, R4.2
- new net N$6: IC3.TXD, OK1.C
- new net N$8: IC3.RXD, OK2.VO, R6.1
- new net N$9: OK2.A, R8.1
- new net N.C.: X1G$1.4
- new net RESET_AVR: OK5.VO, R9.2
- new net RX_AVR: OK1.VO, R7.1
- new net TX_AVR: OK2.C
- new net USB_DATA+: IC3.USBDP, X1G$1.3
- new net USB_DATA-: IC3.USBDM, X1G$1.2
- new net VCCINT: C11.2, C13.2, C14.2, IC3.VCC, IC3.VCCIO, OK2.VCC, OK2.VE, OK3.A, OK4.A, R4.1, R5.1, R6.2, X1G$1.1
- net +5V: now also IC2P.VCC, LED1_BOTTOM.A, LED2_BOTTOM.A, OK1.VCC, OK1.VE, OK5.VCC, OK5.VE, R7.2, R8.2, R9.1
- net GND: now also OK1.GND, OK3.EMIT, OK5.GND, R14.2
Other:
- note added: "00"
